Commit message: Add files via upload

File: articubot_one/description/arm.xacro (robot description, xacro)
@@ -161,5 +161,5 @@
             <origin xyz="0 0 0" rpy="0 0 0"/>
             <geometry>
-                <box size="0.04 0.4 0.01"/>
+                <box size="0.04 0.6 0.01"/>
             </geometry>
             <material name="red"/>
@@ -168,5 +168,5 @@
             <origin xyz="0 0 0" rpy="0 0 0"/>
             <geometry>
-                <box size="0.04 0.4 0.01"/>
+                <box size="0.04 0.6 0.01"/>
             </geometry>
         </collision>
@@ -186,19 +186,19 @@
         <origin xyz="0 0 0" rpy="0 0 0"/>
         <axis xyz="0 1 0"/>
-        <limit lower="0.02" upper="0.2" effort="100" velocity="0.1"/>
+        <limit lower="0.02" upper="0.3" effort="100" velocity="0.1"/>
         <dynamics damping="1" friction="2" />
     </joint>
     <link name="finger">
         <visual>
-            <origin xyz="0 0 0.1" rpy="0 0 0"/>
-            <geometry>
-                <box size="0.04 0.04 0.2"/>
-            </geometry>
-            <material name="blue"/>
-        </visual>
-        <collision>
-            <origin xyz="0 0 0.1" rpy="0 0 0"/>
-            <geometry>
-                <box size="0.04 0.04 0.2"/>
+            <origin xyz="0 0 0.3" rpy="0 0 0"/>
+            <geometry>
+                <box size="0.04 0.04 0.6"/>
+            </geometry>
+            <material name="blue"/>
+        </visual>
+        <collision>
+            <origin xyz="0 0 0.3" rpy="0 0 0"/>
+            <geometry>
+                <box size="0.04 0.04 0.8"/>
             </geometry>
         </collision>
@@ -212,19 +212,19 @@
         <origin xyz="0 0 0" rpy="0 0 0"/>
         <axis xyz="0 1 0"/>
-        <limit lower="-0.02" upper="-0.2" effort="100" velocity="0.1"/>
+        <limit lower="-0.02" upper="-0.3" effort="100" velocity="0.1"/>
         <dynamics damping="1" friction="2" />
     </joint>
     <link name="finger1">
         <visual>
-            <origin xyz="0 0 0.1" rpy="0 0 0"/>
-            <geometry>
-                <box size="0.04 0.04 0.2"/>
-            </geometry>
-            <material name="blue"/>
-        </visual>
-        <collision>
-            <origin xyz="0 0 0.1" rpy="0 0 0"/>
-            <geometry>
-                <box size="0.04 0.04 0.2"/>
+            <origin xyz="0 0 0.3" rpy="0 0 0"/>
+            <geometry>
+                <box size="0.04 0.04 0.6"/>
+            </geometry>
+            <material name="blue"/>
+        </visual>
+        <collision>
+            <origin xyz="0 0 0.3" rpy="0 0 0"/>
+            <geometry>
+                <box size="0.04 0.04 0.8"/>
             </geometry>
         </collision>

File: articubot_one/description/robot.urdf.xacro (robot description, xacro)
@@ -6,4 +6,5 @@
     <xacro:include filename="cart.xacro" />
     <xacro:include filename="arm.xacro" />
+    <xacro:include filename="lidar.xacro" />
     <xacro:include filename="arm_tr.xacro" />
     <xacro:include filename="arm1_tr.xacro" />
